Commit message: Update my_robot.xacro file to include sensors

File: src/my_robot/urdf/my_robot.xacro (robot description, xacro)
@@ -23,4 +23,60 @@
     <dynamics damping="1.0" friction="1.0"/>
   </joint>
+  <joint type="fixed" name="camera_joint">
+  	<origin xyz="0.2 0 0" rpy="0 0 0"/>
+    <child link="camera" />
+    <parent link="chassis" />
+    <axis xyz="0 1 0" rpy="0 0 0"/>
+  </joint>
+  <joint type="fixed" name="hokuyo_joint">
+  	<origin xyz="0.15 0 0.1" rpy="0 0 0" />
+    <child link="hokuyo" />
+    <parent link="chassis" />
+    <axis xyz="0 1 0" />
+  </joint>
+  <link name="hokuyo">
+  	<inertial>
+    	<origin xyz="0 0 0" rpy="0 0 0" />
+        <mass value="1e-5"/>
+        <inertia
+        	ixx="1e-6" ixy="0" ixz="0"
+        	iyy="1e-6" iyz="0"
+            izz="1e-6"/>
+    </inertial>
+    <visual name="hokuyo_visual">
+    	<origin xyz="0 0 0" rpy="0 0 0" />
+        <geometry>
+        	<mesh filename="package://my_robot/meshes/hokuyo.dae" />
+        </geometry>
+    </visual>
+    <collision name="hokuyo_collision">
+    	<origin xyz="0 0 0" rpy="0 0 0" />
+        <geometry>
+        	<box size="0.1 0.1 0.1" />
+        </geometry>
+    </collision>
+  </link>
+  <link name="camera">
+  	<inertial>
+    	<origin xyz="0.05 0.05 0.05" />
+        <mass value="0.1"/>
+        <inertia
+        	ixx="1e-6" ixy="0" ixz="0"
+            iyy="1e-6" iyz="0"
+            izz="1e-6"/>
+    </inertial>
+  	<visual name="camera_visual">
+    	<origin xyz="0 0 0" rpy="0 0 0" />
+    	<geometry>
+        	<box size="0.05 0.05 0.05"/>
+        </geometry>
+    </visual>
+    <collision name="camera_collision">
+    	<origin xyz="0 0 0" rpy="0 0 0" />
+    	<geometry>
+        	<box size="0.05 0.05 0.05"/>
+        </geometry>
+    </collision>
+  </link>
   <link name="left_wheel">
   	<inertial>

Commit message: Add rivitz integration

File: src/my_robot/urdf/my_robot.xacro (robot description, xacro)
@@ -1,4 +1,5 @@
 <?xml version='1.0'?>
 <robot name="my_robot" xmlns:xacro="http://www.ros.org/wiki/xacro">
+<xacro:include filename="$(find my_robot)/urdf/my_robot.gazebo" />
   <link name="robot_footprint"></link>
   <joint name="robot_footprint_joint" type="fixed">
@@ -171,3 +172,12 @@
     </visual>
   </link>
+  <gazebo reference="left_wheel">
+    <material>Gazebo/Green</material>
+  </gazebo>
+  <gazebo reference="right_wheel">
+    <material>Gazebo/Green</material>
+  </gazebo>
+  <gazebo reference="chassis">
+    <material>Gazebo/Red</material>
+  </gazebo>
 </robot>

Commit message: map_my_world

File: src/my_robot/urdf/my_robot.xacro (robot description, xacro)
@@ -36,4 +36,11 @@
     <axis xyz="0 1 0" />
   </joint>
+  <joint name="camera_optical_joint" type="fixed">
+    <origin xyz="0 0 0" rpy="-1.5707 0 -1.5707"/>
+    <parent link="camera"/>
+    <child link="camera_link_optical"/>
+  </joint>
+  <link name="camera_link_optical">
+  </link>
   <link name="hokuyo">
   	<inertial>
